File: Kicad/full_digit.sch (KiCad schematic (older format))
At the start: 54 parts, among them J1 CONN_8, J2 CONN_8, J3 CONN_8, J4 CONN_8, T1 TP, T10 TP, T11 TP, T12 TP, T13 TP, T14 TP, T15 TP, T16 TP, T17 TP, T2 TP, T3 TP, T4 TP, T5 TP, T6 TP, T7 TP, T8 TP, T9 TP, U1 TLC5917, X1 MTHOLE, X2 MTHOLE, X3 MTHOLE, X4 MTHOLE

Commit message: Fix Inter-board Connector
This fixes the inter-board connector polarity issue (#2) in the
schematic.
Parts:
- removed C3, C4: 4.7uF, ~, symbol C
- removed T1, T2, T3, T4, T5, T6, T7, T8, T9: TP, symbol TP
- added J5, J6, J7, J8: CONN_8, symbol CONN_8
- renumbered C5 to C3, J4 to J3, J3 to J4, T10 to T0, T11 to T1, T12 to T2, T13 to T3, T14 to T4, T15 to T5, T16 to T6, T17 to T7
Connections:
- wire segments 85 -> 80
Other:
- moved on the sheet: C1, C2, C3, D1, D10, D11, D12, D13, D14, D15, D16, D17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

Commit message: +5V to Vcc
Fix for Issue +13 in schematic.
Connections:
- net labels added: VCC
- net labels removed: +5V
Other:
- note added: "Vcc can be between 3.0 and 5.5 V. \nComms should match Vcc."
Changed lines of the file:
@@
-$EndComp
-$Comp
-L +5V #PWR02
-U 1 1 541DFC76
-P 6050 2950
-F 0 "#PWR02" H 6050 3040 20  0001 C CNN
-F 1 "+5V" H 6050 3040 30  0000 C CNN
-F 2 "" H 6050 2950 60  0000 C CNN
-F 3 "" H 6050 2950 60  0000 C CNN
-	1    6050 2950
-	1    0    0    -1
 $EndComp
 $Comp
@@
 F 3 "" H 2150 1050 60  0000 C CNN
 	1    2150 1050
-	1    0    0    -1
-$EndComp
-$Comp
-L +5V #PWR04
-U 1 1 541DFDAF
-P 2350 1050
-F 0 "#PWR04" H 2350 1140 20  0001 C CNN
-F 1 "+5V" H 2350 1140 30  0000 C CNN
-F 2 "" H 2350 1050 60  0000 C CNN
-F 3 "" H 2350 1050 60  0000 C CNN
-	1    2350 1050
 	1    0    0    -1
 $EndComp
@@
 $EndComp
 $Comp
-L +5V #PWR06
-U 1 1 541E0125
-P 3050 5350
-F 0 "#PWR06" H 3050 5440 20  0001 C CNN
-F 1 "+5V" H 3050 5440 30  0000 C CNN
-F 2 "" H 3050 5350 60  0000 C CNN
-F 3 "" H 3050 5350 60  0000 C CNN
-	1    3050 5350
-	1    0    0    -1
-$EndComp
-$Comp
 L GND #PWR07
 U 1 1 541E0134
@@
 OUT
 $Comp
-L +5V #PWR08
-U 1 1 541E5935
-P 3050 1050
-F 0 "#PWR08" H 3050 1140 20  0001 C CNN
-F 1 "+5V" H 3050 1140 30  0000 C CNN
-F 2 "" H 3050 1050 60  0000 C CNN
-F 3 "" H 3050 1050 60  0000 C CNN
-	1    3050 1050
-	1    0    0    -1
-$EndComp
-$Comp
 L GND #PWR09
 U 1 1 541E5944
@@
 F 3 "" H 2800 5350 60  0000 C CNN
 	1    2800 5350
-	1    0    0    -1
-$EndComp
-$Comp
-L +5V #PWR011
-U 1 1 541E5BFE
-P 2700 5350
-F 0 "#PWR011" H 2700 5440 20  0001 C CNN
-F 1 "+5V" H 2700 5440 30  0000 C CNN
-F 2 "" H 2700 5350 60  0000 C CNN
-F 3 "" H 2700 5350 60  0000 C CNN
-	1    2700 5350
 	1    0    0    -1
 $EndComp
@@
 Wire Wire Line
 	3250 1150 3850 1150
+$Comp
+L VCC #PWR?
+U 1 1 544374B1
+P 6050 2950
+F 0 "#PWR?" H 6050 3050 30  0001 C CNN
+F 1 "VCC" H 6050 3050 30  0000 C CNN
+F 2 "~" H 6050 2950 60  0000 C CNN
+F 3 "~" H 6050 2950 60  0000 C CNN
+	1    6050 2950
+	1    0    0    -1
+$EndComp
+$Comp
+L VCC #PWR?
+U 1 1 54437564
+P 2350 1050
+F 0 "#PWR?" H 2350 1150 30  0001 C CNN
+F 1 "VCC" H 2350 1150 30  0000 C CNN
+F 2 "~" H 2350 1050 60  0000 C CNN
+F 3 "~" H 2350 1050 60  0000 C CNN
+	1    2350 1050
+	1    0    0    -1
+$EndComp
+$Comp
+L VCC #PWR?
+U 1 1 5443757D
+P 3050 1050
+F 0 "#PWR?" H 3050 1150 30  0001 C CNN
+F 1 "VCC" H 3050 1150 30  0000 C CNN
+F 2 "~" H 3050 1050 60  0000 C CNN
+F 3 "~" H 3050 1050 60  0000 C CNN
+	1    3050 1050
+	1    0    0    -1
+$EndComp
+$Comp
+L VCC #PWR?
+U 1 1 5443758C
+P 3050 5350
+F 0 "#PWR?" H 3050 5450 30  0001 C CNN
+F 1 "VCC" H 3050 5450 30  0000 C CNN
+F 2 "~" H 3050 5350 60  0000 C CNN
+F 3 "~" H 3050 5350 60  0000 C CNN
+	1    3050 5350
+	1    0    0    -1
+$EndComp
+$Comp
+L VCC #PWR?
+U 1 1 5443759B
+P 2700 5350
+F 0 "#PWR?" H 2700 5450 30  0001 C CNN
+F 1 "VCC" H 2700 5450 30  0000 C CNN
+F 2 "~" H 2700 5350 60  0000 C CNN
+F 3 "~" H 2700 5350 60  0000 C CNN
+	1    2700 5350
+	1    0    0    -1
+$EndComp
+Text Notes 5200 2600 0    60   ~ 0
+Vcc can be between 3.0 and 5.5 V. \nComms should match Vcc.
 $EndSCHEMATC

Commit message: Added fuses
Added two PTC resettable fuses, one to each input terminal. This
resolves issue #3. The extra resistance is a maximum of 50 mOhm per PTC
under normal conditions. This reduces the maximum number of series
panels from 25 to 17 between additional power connectors are needed. The
trip current is 3 A.
Parts:
- added PTC? (x2): 3A, ~, symbol PTC
Connections:
- wire segments 80 -> 82
Other:
- moved on the sheet: C2, C3, J1, J2, J3, J4, J5, J6, J7, J8

Commit message: Updated Decoupling Capacitors
Updated the decoupling capacitors and consolidated C2-C5 into C2. One
4.7uF cap should be enough to ensure that the voltage drop resulting
from all segments off to all segments on remains less than 1 V while the
power supply compensates. C1 decouples U1, which has a maximum clock
frequency of 30 MHz, but will be operating well under that for most
applications. One standard 0.1uF cap on the Vcc rail should be enough.
Parts:
- removed C3: 4.7uF, ~, symbol C
- C1: value 0.1uF -> 0.1uF 12V
- C2: value 4.7uF -> 4.7uF 25V
- PTC? (x2): value 3A -> 0ZCF0300AF2C
Connections:
- wire segments 82 -> 81
Changed lines of the file:
@@
 Title "Full Digit"
 Date "19 oct 2014"
-Rev "1"
+Rev "2"
 Comp ""
 Comment1 ""
@@
 P 5450 3350
 F 0 "C1" H 5450 3450 40  0000 L CNN
-F 1 "0.1uF" H 5456 3265 40  0000 L CNN
+F 1 "0.1uF 12V" H 5456 3265 40  0000 L CNN
 F 2 "~" H 5488 3200 30  0000 C CNN
 F 3 "~" H 5450 3350 60  0000 C CNN
@@
 $EndComp
 $Comp
-L C C3
-U 1 1 542273B0
-P 2550 5750
-F 0 "C3" H 2550 5850 40  0000 L CNN
-F 1 "4.7uF" H 2556 5665 40  0000 L CNN
-F 2 "~" H 2588 5600 30  0000 C CNN
-F 3 "~" H 2550 5750 60  0000 C CNN
-	1    2550 5750
-	1    0    0    -1
-$EndComp
-$Comp
-L GND #PWR013
-U 1 1 542273BF
-P 2550 6050
-F 0 "#PWR013" H 2550 6050 30  0001 C CNN
-F 1 "GND" H 2550 5980 30  0001 C CNN
-F 2 "~" H 2550 6050 60  0000 C CNN
-F 3 "~" H 2550 6050 60  0000 C CNN
-	1    2550 6050
-	1    0    0    -1
-$EndComp
-$Comp
 L C C2
 U 1 1 54228938
 P 3050 1650
 F 0 "C2" H 3050 1750 40  0000 L CNN
-F 1 "4.7uF" H 3056 1565 40  0000 L CNN
+F 1 "4.7uF 25V" H 3056 1565 40  0000 L CNN
 F 2 "~" H 3088 1500 30  0000 C CNN
 F 3 "~" H 3050 1650 60  0000 C CNN
@@
 	5450 3150 5450 3050
 Connection ~ 6050 3050
-Wire Wire Line
-	2550 6050 2550 5950
 Connection ~ 6900 1500
 Wire Wire Line
@@
 Wire Wire Line
 	2550 5550 2550 5350
-Connection ~ 2550 5550
 Connection ~ 3850 5550
 Wire Wire Line
@@
 P 2250 1150
 F 0 "PTC?" V 2400 1200 50  0000 C CNN
-F 1 "3A" V 2500 1250 50  0000 C CNN
+F 1 "0ZCF0300AF2C" V 2500 1250 50  0000 C CNN
 F 2 "~" H 2250 1150 60  0000 C CNN
 F 3 "~" H 2250 1150 60  0000 C CNN
@@
 P 3500 5550
 F 0 "PTC?" V 3350 5600 50  0000 C CNN
-F 1 "3A" V 3250 5600 50  0000 C CNN
+F 1 "0ZCF0300AF2C" V 3250 5600 50  0000 C CNN
 F 2 "~" H 3500 5550 60  0000 C CNN
 F 3 "~" H 3500 5550 60  0000 C CNN

Commit message: Updated Footprints for Rev 2
Parts:
- gave numbers to parts that had none: 2
Changed lines of the file:
@@
 Sheet 1 1
 Title "Full Digit"
-Date "19 oct 2014"
+Date "21 oct 2014"
 Rev "2"
 Comp ""
@@
 $EndComp
 $Comp
-L GND #PWR03
+L GND #PWR02
 U 1 1 541DFCB0
 P 5750 4250
-F 0 "#PWR03" H 5750 4250 30  0001 C CNN
+F 0 "#PWR02" H 5750 4250 30  0001 C CNN
 F 1 "GND" H 5750 4180 30  0001 C CNN
 F 2 "" H 5750 4250 60  0000 C CNN
@@
 $EndComp
 $Comp
-L GND #PWR05
+L GND #PWR03
 U 1 1 541DFE24
 P 2650 1950
-F 0 "#PWR05" H 2650 1950 30  0001 C CNN
+F 0 "#PWR03" H 2650 1950 30  0001 C CNN
 F 1 "GND" H 2650 1880 30  0001 C CNN
 F 2 "" H 2650 1950 60  0000 C CNN
@@
 $EndComp
 $Comp
-L VLED #PWR16
+L VLED #PWR17
 U 1 1 541E0116
 P 2550 5350
-F 0 "#PWR16" H 2550 5550 40  0001 C CNN
+F 0 "#PWR17" H 2550 5550 40  0001 C CNN
 F 1 "VLED" H 2550 5500 40  0000 C CNN
 F 2 "" H 2550 5350 60  0000 C CNN
@@
 $EndComp
 $Comp
-L GND #PWR07
+L GND #PWR04
 U 1 1 541E0134
 P 2600 4950
-F 0 "#PWR07" H 2600 4950 30  0001 C CNN
+F 0 "#PWR04" H 2600 4950 30  0001 C CNN
 F 1 "GND" H 2600 4880 30  0001 C CNN
 F 2 "" H 2600 4950 60  0000 C CNN
@@
 OUT
 $Comp
-L GND #PWR09
+L GND #PWR05
 U 1 1 541E5944
 P 3750 1950
-F 0 "#PWR09" H 3750 1950 30  0001 C CNN
+F 0 "#PWR05" H 3750 1950 30  0001 C CNN
 F 1 "GND" H 3750 1880 30  0001 C CNN
 F 2 "" H 3750 1950 60  0000 C CNN
@@
 SDO
 $Comp
-L GND #PWR010
+L GND #PWR06
 U 1 1 541E5BE0
 P 2350 4950
-F 0 "#PWR010" H 2350 4950 30  0001 C CNN
+F 0 "#PWR06" H 2350 4950 30  0001 C CNN
 F 1 "GND" H 2350 4880 30  0001 C CNN
 F 2 "" H 2350 4950 60  0000 C CNN
@@
 $EndComp
 $Comp
-L VLED #PWR15
+L VLED #PWR16
 U 1 1 541E5BEF
 P 2400 5350
-F 0 "#PWR15" H 2400 5550 40  0001 C CNN
+F 0 "#PWR16" H 2400 5550 40  0001 C CNN
 F 1 "VLED" H 2400 5500 40  0000 C CNN
 F 2 "" H 2400 5350 60  0000 C CNN
@@
 $EndComp
 $Comp
-L GND #PWR012
+L GND #PWR07
 U 1 1 54226A7E
 P 5450 3650
-F 0 "#PWR012" H 5450 3650 30  0001 C CNN
+F 0 "#PWR07" H 5450 3650 30  0001 C CNN
 F 1 "GND" H 5450 3580 30  0001 C CNN
 F 2 "~" H 5450 3650 60  0000 C CNN
@@
 $EndComp
 $Comp
-L GND #PWR016
+L GND #PWR08
 U 1 1 54228BB7
 P 3050 1950
-F 0 "#PWR016" H 3050 1950 30  0001 C CNN
+F 0 "#PWR08" H 3050 1950 30  0001 C CNN
 F 1 "GND" H 3050 1880 30  0001 C CNN
 F 2 "~" H 3050 1950 60  0000 C CNN
@@
 $EndComp
 $Comp
-L GND #PWR017
+L GND #PWR09
 U 1 1 542399CF
 P 8150 5750
-F 0 "#PWR017" H 8150 5750 30  0001 C CNN
+F 0 "#PWR09" H 8150 5750 30  0001 C CNN
 F 1 "GND" H 8150 5680 30  0001 C CNN
 F 2 "~" H 8150 5750 60  0000 C CNN
@@
 	3750 1150 4350 1150
 $Comp
-L VCC #PWR?
+L VCC #PWR010
 U 1 1 544374B1
 P 6050 2950
-F 0 "#PWR?" H 6050 3050 30  0001 C CNN
+F 0 "#PWR010" H 6050 3050 30  0001 C CNN
 F 1 "VCC" H 6050 3050 30  0000 C CNN
 F 2 "~" H 6050 2950 60  0000 C CNN
@@
 $EndComp
 $Comp
-L VCC #PWR?
+L VCC #PWR011
 U 1 1 54437564
 P 2850 1050
-F 0 "#PWR?" H 2850 1150 30  0001 C CNN
+F 0 "#PWR011" H 2850 1150 30  0001 C CNN
 F 1 "VCC" H 2850 1150 30  0000 C CNN
 F 2 "~" H 2850 1050 60  0000 C CNN
@@
 $EndComp
 $Comp
-L VCC #PWR?
+L VCC #PWR012
 U 1 1 5443757D
 P 3550 1050
-F 0 "#PWR?" H 3550 1150 30  0001 C CNN
+F 0 "#PWR012" H 3550 1150 30  0001 C CNN
 F 1 "VCC" H 3550 1150 30  0000 C CNN
 F 2 "~" H 3550 1050 60  0000 C CNN
@@
 $EndComp
 $Comp
-L VCC #PWR?
+L VCC #PWR013
 U 1 1 5443758C
 P 2650 5350
-F 0 "#PWR?" H 2650 5450 30  0001 C CNN
+F 0 "#PWR013" H 2650 5450 30  0001 C CNN
 F 1 "VCC" H 2650 5450 30  0000 C CNN
 F 2 "~" H 2650 5350 60  0000 C CNN
@@
 $EndComp
 $Comp
-L VCC #PWR?
+L VCC #PWR014
 U 1 1 5443759B
 P 2300 5350
-F 0 "#PWR?" H 2300 5450 30  0001 C CNN
+F 0 "#PWR014" H 2300 5450 30  0001 C CNN
 F 1 "VCC" H 2300 5450 30  0000 C CNN
 F 2 "~" H 2300 5350 60  0000 C CNN
@@
 Vcc can be between 3.0 and 5.5 V. \nComms should match Vcc.
 $Comp
-L PTC PTC?
+L PTC PTC1
 U 1 1 54437841
 P 2250 1150
-F 0 "PTC?" V 2400 1200 50  0000 C CNN
+F 0 "PTC1" V 2400 1200 50  0000 C CNN
 F 1 "0ZCF0300AF2C" V 2500 1250 50  0000 C CNN
 F 2 "~" H 2250 1150 60  0000 C CNN
@@
 $EndComp
 $Comp
-L PTC PTC?
+L PTC PTC2
 U 1 1 54437850
 P 3500 5550
-F 0 "PTC?" V 3350 5600 50  0000 C CNN
+F 0 "PTC2" V 3350 5600 50  0000 C CNN
 F 1 "0ZCF0300AF2C" V 3250 5600 50  0000 C CNN
 F 2 "~" H 3500 5550 60  0000 C CNN
