File: Kicad/half_digit/half_digit.sch (KiCad schematic (older format))
At the start: 33 parts, among them J1 CONN_8, J2 CONN_8, J3 CONN_8, J4 CONN_8, J5 SPARK, J6 BARREL_JACK, U1 TLC5917, U2 AOZ1280

Commit message: Partial Layout
LEDs, inter-board connectors, and buck converter placed. Still need to
figure out placement of DC jack.
Parts:
- added C4: 0.1uF, ~, symbol C
- added J5, J6: CONN_12, symbol CONN_12
- added X1, X2, X3, X4: MTHOLE, ~, symbol MTHOLE
- R2: value 10k -> 9.53k 1%
- renumbered J6 to J7, J5 to U3
Connections:
- wire segments 93 -> 96
- no-connect marks 16 -> 32
Other:
- moved on the sheet: C1, C2, C3, D16, J7, L1, PTC1, R2, R3, R4, U2

Commit message: Rough draft of half digit layout
Parts:
- removed U3: SPARK, symbol SPARK
- added J7, J8: CONN_12, symbol CONN_12
- renumbered J7 to J9
Connections:
- wire segments 96 -> 111
- no-connect marks 32 -> 2
Other:
- note added: "A0"
- note added: "D0"
- note added: "Spark Core"
- note added: "VCC"
- note added: "VIN"
- moved on the sheet: J1, J2, J3, J4, J5, J6
